Commit message: [description] Add wheel properties

File: four_wheel_steering_description/urdf/vehicle.urdf.xacro (robot description, xacro)
@@ -8,5 +8,4 @@
   <xacro:include filename="$(find four_wheel_steering_description)/urdf/sensors.xacro" />
   <!-- Base Properties -->
-  <xacro:property name="mass_base" value="500" />
   <xacro:property name="base_x_size" value="1.66000" />
   <xacro:property name="base_y_size" value="0.60000" />
@@ -14,4 +13,10 @@
   <xacro:property name="wheelbase" value="2" />
   <xacro:property name="track" value="1.1" />
+  <xacro:property name="mass_base" value="500" />
+  <!-- Wheel Properties -->
+  <xacro:property name="steering_link_mass" value="30" />
+  <xacro:property name="mass_wheel" value="5" />
+  <xacro:property name="wheel_length" value="0.2" />
+  <xacro:property name="wheel_radius" value="0.45" />
   <!-- Wheel Mounting Positions -->
   <xacro:property name="ground_clearance" value="0.35" />

File: four_wheel_steering_description/urdf/wheel.xacro (robot description, xacro)
@@ -1,5 +1,4 @@
 <?xml version="1.0"?>
 <robot xmlns:xacro="http://www.ros.org/wiki/xacro" name="wheel">
-  <!--<xacro:property name="M_PI" default="3.14159"/>-->
   <!-- Wheel Properties -->
   <xacro:property name="wheel_length" value="0.2" />

Commit message: [description] Turn wheel joint instead of link

File: four_wheel_steering_description/urdf/vehicle.urdf.xacro (robot description, xacro)
@@ -50,5 +50,5 @@
       <!-- visual wheel -->
       <visual>
-        <origin xyz="0 0 0" rpy="${M_PI/2} 0 0" />
+        <origin xyz="0 0 0" rpy="0 0 0" />
         <geometry>
           <cylinder length="${wheel_length}" radius="${wheel_radius}"/>

File: four_wheel_steering_description/urdf/wheel.xacro (robot description, xacro)
@@ -12,5 +12,5 @@
       <inertial>
         <mass value="${mass_wheel}" />
-        <origin xyz="0 0 0" rpy="${M_PI/2} 0 0" />
+        <origin xyz="0 0 0" rpy="0 0 0" />
         <inertia  ixx="${mass_wheel/4.0*(wheel_radius*wheel_radius+wheel_length*wheel_length/3.0)}" ixy="0" ixz="0"
                   iyy="${mass_wheel/4.0*(wheel_radius*wheel_radius+wheel_length*wheel_length/3.0)}" iyz="0"
@@ -19,5 +19,5 @@
       <xacro:insert_block name="visual_wheel"/>
       <collision>
-        <origin xyz="0 0 0" rpy="${M_PI/2} 0 0" />
+        <origin xyz="0 0 0" rpy="0 0 0" />
         <geometry>
           <cylinder length="${wheel_length}" radius="${wheel_radius}" />
@@ -35,5 +35,5 @@
       <child link="${wheel_prefix}_wheel_link"/>
       <xacro:insert_block name="joint_origin"/>
-      <axis xyz="0 1 0" rpy="0 0 0" />
+      <axis xyz="0 0 1" rpy="0 0 0" />
     </joint>
     <transmission name="${wheel_prefix}_wheel_trans" type="SimpleTransmission">

File: four_wheel_steering_description/urdf/wheel_steered.xacro (robot description, xacro)
@@ -35,5 +35,5 @@
     </transmission>
     <xacro:wheel wheel_prefix="${wheel_prefix}" parent_link="${wheel_prefix}_steering" left_right="${left_right}">
-      <origin xyz="0 ${wheel_origin_y} 0" rpy="0 0 0" />
+      <origin xyz="0 ${wheel_origin_y} 0" rpy="${-M_PI/2} 0 0" />
       <xacro:insert_block name="visual_wheel"/>
     </xacro:wheel>

Commit message: [description] reduce urdf visual box

File: four_wheel_steering_description/urdf/vehicle.urdf.xacro (robot description, xacro)
@@ -39,24 +39,7 @@
       </visual>
       <!-- visual steering -->
-      <visual>
-        <origin xyz="0 0 0" rpy="0 0 0"/>
-        <geometry>
-          <box size="0.05 ${steering_link_y} 0.05"/>
-        </geometry>
-        <material name="blue">
-          <color rgba="0.2 0.2 0.6 1"/>
-        </material>
-      </visual>
+      <box size="0.05 ${steering_link_y} 0.05"/>
       <!-- visual wheel -->
-      <visual>
-        <origin xyz="0 0 0" rpy="0 0 0" />
-        <geometry>
-          <cylinder length="${wheel_length}" radius="${wheel_radius}"/>
-          <!--<mesh filename="package://four_wheel_steering_description/meshes/wheel.dae"/>-->
-        </geometry>
-        <material name="black">
-          <color rgba="0 0 0 1"/>
-        </material>
-      </visual>
+      <cylinder length="${wheel_length}" radius="${wheel_radius}"/>
     </xacro:chassis>
     <xacro:sensors/>

File: four_wheel_steering_description/urdf/wheel.xacro (robot description, xacro)
@@ -17,5 +17,13 @@
                   izz="${mass_wheel*wheel_radius*wheel_radius/2.0}" />
       </inertial>
-      <xacro:insert_block name="visual_wheel"/>
+      <visual>
+        <origin xyz="0 0 0" rpy="0 0 0" />
+        <geometry>
+          <xacro:insert_block name="visual_wheel"/>
+        </geometry>
+        <material name="black">
+          <color rgba="0 0 0 1"/>
+        </material>
+      </visual>
       <collision>
         <origin xyz="0 0 0" rpy="0 0 0" />

File: four_wheel_steering_description/urdf/wheel_steered.xacro (robot description, xacro)
@@ -7,5 +7,13 @@
   <xacro:macro name="wheel_steered" params="wheel_prefix parent_link wheel_origin_y left_right *joint_origin *visual_steering *visual_wheel">
     <link name="${wheel_prefix}_steering">
-      <xacro:insert_block name="visual_steering"/>
+      <visual>
+        <origin xyz="0 0 0" rpy="0 0 ${left_right * M_PI/2 - M_PI/2}"/>
+        <geometry>
+          <xacro:insert_block name="visual_steering"/>
+        </geometry>
+        <material name="blue">
+          <color rgba="0.2 0.2 0.6 1"/>
+        </material>
+      </visual>
       <inertial>
         <mass value="${steering_link_mass}" />
